File: Hardware/ServoLess/ServoLess.kicad_pcb (KiCad board)
At the start: 4 copper layers, 46 x 46 mm, 98 parts, among them J1 XT30PW-M, J2 USB_C_Receptacle_USB2.0, J3 Conn_01x02_MountingPin, J4 Conn_01x03_MountingPin, J6 Conn_01x04_MountingPin, SW1 SW_Push, SW2 SW_Push, U1 S8050, U10 INA240A2PW, U11 INA240A2PW, U12 AS5048A, U2 S8050, U3 ESP32-S3FN8, U4 CH343P, U5 TPS54202DDC, U6 SPX3819M5-L-3-3, U7 AMS1117-3.3, U8 TJA1050T, U9 DRV8313PWP, Y1 Crystal_GND24

Commit message: ServoLess v2
Other:
- board text added: "Ver 1.1"
- board text removed: "Ver 2.0"
